File: pcb/packaged-amp/packaged-amp.kicad_pcb (KiCad board)
At the start: 4 copper layers, 56.6 x 82.7 mm, 70 parts, among them J7 Conn_Coaxial, J8 USB_B, U1 TLV2172, U2 OPA2822, U4 MC78L06F-TP, U5 MC79L06F-TP

Commit message: next revision
Parts:
- removed R11: 470, Resistor_SMD:R_0603_1608Metric
- removed the R12 at (119.0, 86.8)
- removed TP11, TP12: DNP, TestPoint:TestPoint_Pad_4.0x4.0mm
- added C22: 47p, Capacitor_SMD:C_0603_1608Metric, F.Cu at (125.5, 96.5)
- added J2: Conn_Coaxial, Connector_Coaxial:U.FL_Hirose_U.FL-R-SMT-1_Vertical, F.Cu at (109.2, 118.8)
- added R13: 1.2k, Resistor_SMD:R_0603_1608Metric, F.Cu at (123.7, 93.2)
- added R14: 169, Resistor_SMD:R_0603_1608Metric, F.Cu at (113.7, 92.8)
- added R15: 220, Resistor_SMD:R_0603_1608Metric, F.Cu at (113.7, 89.5)
- added RV2: 200, Potentiometer_SMD:Potentiometer_Bourns_3314G_Vertical, F.Cu at (118.7, 91.2)
- C10: renamed from C1; value DNP -> 10p
- C11: value 12-60p -> DNP
- C6: renamed from C9; value 100p -> 180p
- C8: renamed from C10; value DNP -> 10p
- F1: footprint Fuse:Fuse_1206_3216Metric -> Fuse:Fuse_0603_1608Metric
- L1: value DLW5BTM102SQ2L -> DLW5BTM142SQ2L
- L2, L3, L4: value 10u -> 6.8u
- R3: renamed from R5; value 360 -> 430
- R8: renamed from R10; value 470 -> 220
- moved NT1 14.3 mm to (122.0, 118.0)
- moved C18 9.83 mm to (123.8, 96.5), turned to -90 degrees
- moved R1 8.50 mm to (120.8, 109.0), turned to 90 degrees
- moved R16 7.25 mm to (118.5, 86.8), turned to 180 degrees
- moved RV1 6.93 mm to (109.8, 106.0)
- moved C14 6.25 mm to (116.5, 104.8)
- moved C3 6.25 mm to (115.0, 97.0)
- moved C4 6.25 mm to (122.0, 100.5)
- moved R2 6.25 mm to (123.5, 104.8)
- moved R3 6.25 mm to (118.2, 104.8)
- moved R4 6.25 mm to (120.0, 104.8)
- moved R5 6.25 mm to (121.8, 104.8)
- moved R6 6.25 mm to (114.8, 104.8)
- moved R8 6.25 mm to (122.0, 96.5)
- moved U2 6.25 mm to (118.5, 98.8)
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- renumbered C5 to C1, C3 to C12, C7 to C13, C8 to C15, C18 to C16, C15 to C17, C19 to C18, C16 to C19, C6 to C2, C28 to C20, C29 to C21, C30 to C23, C31 to C24, C12 to C3, C13 to C4, C4 to C5, C2 to C7, C17 to C9, D11 to D1, D1 to D2, D2 to D3, D6 to D4, J8 to J1, J7 to J3, R8 to R10, R9 to R12, R13 to R16, R25 to R17, R6 to R2, R2 to R4, R3 to R5, R14 to R6, R4 to R7, R7 to R9, TP4 to TP1, TP6 to TP2, U4 to U3, U5 to U4
Connections:
- C10 pad 1: Net-(C1-Pad1) -> Net-(C10-Pad1)
- C10 pad 2: /return_kelvin -> GND
- C11 pad 1: Net-(C1-Pad1) -> GND
- C11 pad 2: /return_kelvin -> Net-(C10-Pad1)
- C6 pad 1: Net-(C1-Pad1) -> Net-(C10-Pad1)
- C6 pad 2: /return_kelvin -> GND
- C8 pad 1: Net-(C1-Pad1) -> Net-(C10-Pad1)
- C8 pad 2: /return_kelvin -> GND
- D2 pad 2: Net-(C1-Pad1) -> Net-(C10-Pad1)
- D3 pad 1: Net-(C1-Pad1) -> Net-(C10-Pad1)
- R1 pad 2: Net-(C1-Pad1) -> Net-(C10-Pad1)
- R2 pad 1: Net-(C1-Pad1) -> Net-(C10-Pad1)
Routing:
- net /return_kelvin: track 54.5 -> 18.5 mm, vias 4 -> 7
- net Net-(C1-Pad1): track 28.0 -> 0.00 mm
- net Net-(C10-Pad1): track 0.00 -> 19.1 mm
- net GND: track 30.4 -> 20.7 mm, vias 92 -> 99
- net Net-(GD1-Pad1): track 11.4 -> 20.6 mm, vias 0 -> 1
- net /out: track 16.5 -> 22.1 mm
- net Net-(R13-Pad1): track 4.51 -> 9.35 mm
- net Net-(R3-Pad1): track 3.32 -> 7.93 mm
- net Net-(C22-Pad1): track 0.00 -> 4.60 mm
- net Net-(E1-Pad2): track 31.1 -> 26.8 mm, vias 4 -> 0
- net Net-(C19-Pad2): track 6.03 -> 9.84 mm
- net Net-(R14-Pad2): track 0.00 -> 2.80 mm
- net Net-(R15-Pad1): track 0.00 -> 2.51 mm
- net Net-(J1-Pad4): track 31.1 -> 28.8 mm
- net Net-(F1-Pad1): track 14.2 -> 15.9 mm
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- added copper zone on F.Cu, net /return_kelvin
Other:
- outline, holes or cut-outs redrawn
- board text added: "5V 0.4A"
- board text added: "Coil"
- board text added: "Comp"
- board text added: "Gain"
- board text added: "Rogowski Coil Amplifier V3.0 2023"
- board text added: "S/N:"
- board text removed: "5V 0.25A"
- board text removed: "Ret"
- board text removed: "Rogowski Coil Amplifier V2.0 2022"
- board text removed: "Sig"

Commit message: first public release
Parts:
- removed E2: SparkGap, wbraun_smd:Spark_Gap
- removed NT1: DNP, NetTie:NetTie-2_SMD_Pad0.5mm
- added J3: Conn_01x01_Female, wbraun_smd:CLIP_ECT81800C036, F.Cu at (114.5, 112.8)
- added J4: Conn_01x01_Female, wbraun_smd:CLIP_ECT81800C036, F.Cu at (104.5, 97.8)
- added J5: Conn_01x01_Female, wbraun_smd:CLIP_ECT81800C036, F.Cu at (124.5, 97.8)
- added J6: Conn_01x01_Female, wbraun_smd:CLIP_ECT81800C036, F.Cu at (114.5, 82.8)
- added R2: 4.7, Resistor_SMD:R_0603_1608Metric, F.Cu at (117.0, 107.8)
- added R3: 4.7, Resistor_SMD:R_0603_1608Metric, F.Cu at (120.0, 107.8)
- added R5: 47, Resistor_SMD:R_0603_1608Metric, F.Cu at (122.2, 103.5)
- C11: footprint wbraun_smd:C_Trimmer_GKG_6mm -> Capacitor_SMD:C_0603_1608Metric
- C5: renamed from C6; value 180p -> 68p
- C7: renamed from C8; value 10p -> 68p
- C9: renamed from C10; value 10p -> 68p
- D3: renamed from D1; value P6SMB6.8CA/TR13 -> 6.8V
- GD1: value GDT_2Pin -> 75V
- J1: renamed from J2; value Conn_Coaxial -> U.FL
- J7: renamed from J3; value Conn_Coaxial -> SMA
- PS1: value A0509S-2WR3 -> A0509S-1WR3
- R19: renamed from R17; value 4.7k -> 2.2k
- R4: renamed from R2; value 47 -> 4.7
- U1: value TLV2172 -> OPA2188
- moved D2 11.0 mm to (115.5, 106.0), turned to 180 degrees
- moved D1 8.62 mm to (118.8, 106.0)
- moved TP2 8.28 mm to (128.5, 110.8)
- moved R1 7.04 mm to (113.8, 109.8), turned to 0 degrees
- moved C11 6.25 mm to (122.2, 106.5), turned to -90 degrees
- moved R4 5.40 mm to (122.2, 110.0)
- moved R18 5.34 mm to (113.2, 85.8)
- moved C22 5.32 mm to (121.5, 93.0), turned to 0 degrees
- moved R15 5.26 mm to (118.5, 93.0), turned to 0 degrees
- moved E1 5.06 mm to (124.5, 118.0), turned to 90 degrees
- moved J1 4.32 mm to (113.5, 118.0)
- moved C17 2.93 mm to (108.8, 91.0)
- moved C19 2.93 mm to (111.0, 88.5)
- moved R10 2.93 mm to (106.8, 91.8), turned to 90 degrees
- moved R12 2.93 mm to (111.0, 91.8)
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- renumbered C9 to C10, C5 to C6, C7 to C8, D2 to D1, D3 to D2, J1 to J2, R7 to R10, R8 to R11, R9 to R12, R10 to R13, R12 to R14, R13 to R15, R14 to R16, R15 to R17, R16 to R18, R3 to R6, R4 to R7, R5 to R8, R6 to R9
Connections:
- C11 pad 2: Net-(C10-Pad1) -> Net-(R4-Pad2)
- C5 pad 1: Net-(C10-Pad1) -> Net-(C5-Pad1)
- C7 pad 1: Net-(C10-Pad1) -> Net-(R3-Pad1)
- C9 pad 1: Net-(C10-Pad1) -> Net-(R3-Pad2)
- D1 pad 2: Net-(C10-Pad1) -> Net-(R3-Pad2)
- D2 pad 1: Net-(C10-Pad1) -> Net-(R3-Pad2)
- J1 pad 2: /return_kelvin -> GND
- R1 pad 2: Net-(C10-Pad1) -> Net-(C5-Pad1)
- R4 pad 1: Net-(C10-Pad1) -> Net-(R3-Pad2)
- R4 pad 2: Net-(R2-Pad2) -> Net-(R4-Pad2)
- U2 pad 3: Net-(R2-Pad2) -> Net-(U2-Pad3)
Routing:
- net GND: track 20.7 -> 50.5 mm, vias 99 -> 137
- net Net-(C10-Pad1): track 19.1 -> 0.00 mm
- net /return_kelvin: track 18.5 -> 0.00 mm, vias 7 -> 0
- net Net-(R3-Pad2): track 0.00 -> 10.8 mm
- net /out: track 22.1 -> 13.8 mm
- net Net-(E1-Pad2): track 26.8 -> 33.9 mm, vias 0 -> 2
- net Net-(U2-Pad3): track 0.00 -> 6.79 mm
- net Net-(R2-Pad2): track 6.59 -> 0.00 mm
- net Net-(R4-Pad2): track 0.00 -> 6.59 mm
- net Net-(R10-Pad1): track 31.5 -> 26.1 mm, vias 2 -> 0
- net Net-(GD1-Pad1): track 20.6 -> 25.0 mm, vias 1 -> 3
- net Net-(R3-Pad1): track 0.00 -> 3.96 mm
- net Net-(C5-Pad1): track 0.00 -> 3.40 mm
- net Net-(R15-Pad2): track 4.60 -> 1.40 mm
- net Net-(U1-Pad1): track 4.10 -> 1.27 mm
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- removed copper zone on F.Cu, net /return_kelvin
Other:
- outline, holes or cut-outs redrawn
- board text added: "Rogowski Coil Amplifier V4.0 2023"
- board text removed: "Rogowski Coil Amplifier V3.0 2023"
