File: pcb/packaged-amp/packaged-amp.kicad_sch (KiCad schematic)
At the start: 105 parts, among them J2 RFShield_TwoPieces, J7 Conn_Coaxial, J8 USB_B, Q1 MMBT3906, Q2 MMBT3904, U1 TLV2172, U2 OPA2822, U3 LMR62014XMF, U4 L78L06_SOT89, U5 L79L05_SOT89

Commit message: finished design of packaged amp
Parts:
- removed D10, D11: LED, wbraun_smd:LED-T1-RIGHT-ANGLE_4.6x4.4mm, symbol Device:LED
- added D10: LED_Dual_KAKA, wbraun_smd:LED_WP934MD, symbol Device:LED_Dual_KAKA
- added TP14: TestPoint, wbraun_smd:THM_MINI, symbol Connector:TestPoint
Connections:
- net GND: now also C7.1; no longer C1.2, C10.2, C11.2, C7.2, C9.2
- net VDD: now also C7.2, D10.2 (K1), D10.4 (K2); no longer C7.1
- net at R28.2: now also D10.1 (A1)
- net return_kelvin: now reaches NT1.1, TP12.1
- net return_kelvin: now also C1.2, C10.2, C11.2, C9.2
- net at F1.2, FB5.1: now also TP14.1
- net at R30.2: now also D10.3 (A2)
- no-connect marks 0 -> 2
Other:
- note added: "Connections for coil"
- note added: "Overload (red)"
- note added: "Power (green)"
- note added: "Simple overload detect circuitry"
- note added: "shield for power supply"
- note removed: "Overload"
- note removed: "Power"
- moved on the sheet: C1, C10, C11, C12, C13, C14, C15, C16, C17, C18, C19, C20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

Commit message: design sent to fab
Parts:
- added D11: SMAJ6.0A-13-F, Diode_SMD:D_SMA, symbol Device:D_Zener
- added E1, E2: SparkGap, wbraun_smd:Spark_Gap, symbol Device:SparkGap
- added GD1: GDT_2Pin, wbraun_smd:GDT_1812, symbol wbraun_ic_lib:GDT_2pin
- added NT2: NetTie_2, NetTie:NetTie-2_SMD_Pad0.5mm, symbol Device:NetTie_2
- C10, C19: MPN (none) -> CL10C220JB81PNC
- C11: MPN (none) -> JZ400
- C12, C13, C5, C6, C7, C8: MPN (none) -> CL10B474KA8NFNC
- C14: MPN (none) -> CL10C330JB8NNNC
- C20, C23, C25, C27, C28, C29, C30, C31: MPN (none) -> CL31A106KAHNNNE
- C22: value 470p -> 330p; MPN (none) -> CL10C330JB8NNNC
- C33, C34: value C -> 0.47u; MPN (none) -> CL10B474KA8NFNC
- C9: MPN (none) -> CL10C151JB8NFNC
- D3, D4, D5: MPN (none) -> PD3S140-7
- FB3, FB4, FB5: MPN (none) -> 742792040
- J2: MPN (none) -> MS288-10F
- J7: MPN (none) -> RF2-49B-T-00-50-G-HDW
- L1: MPN (none) -> VLCF4020T-100MR85
- L2: value L_Ferrite_Coupled -> DLW5BTM142SQ2L; MPN (none) -> DLW5BTM142SQ2L
- R1, R13: MPN (none) -> RMCF1206FT47R0
- R10: MPN (none) -> RMCF0603FT220R
- R11, R12, R20, R21, R8: MPN (none) -> RMCF0603FT2K00
- R14: MPN (none) -> ERJ-3GEY0R00V
- R15, R18: MPN (none) -> RMCF0603FT75K0
- R16: MPN (none) -> RMCF0603FT13K3
- R19: value R -> 0; MPN (none) -> RMCF0805ZT0R00
- R2, R28, R30: MPN (none) -> RMCF0603FT4K70
- R22, R23, R27, R4, R7: MPN (none) -> RMCF0603FT47K0
- R24, R29, R6: MPN (none) -> RMCF0603FG22K0
- R25, R26: MPN (none) -> RMCF0603FG1M00
- R3, R9: MPN (none) -> RMCF0603FT10K0
- R31, R32: value 0 -> 0.1; MPN (none) -> KDV06FR100ET
- R5: MPN (none) -> RC0603FR-07365RL
- RV1: MPN (none) -> PVG3A201C01R00
- U1: MPN (none) -> TLV2172IDR
- U2: MPN (none) -> OPA2822U
- U3: MPN (none) -> LMR62014XMF/NOPB
- U4: value L78L06_SOT89 -> MC78L06F-TP; MPN (none) -> MC78L06F-TP
- U5: value L79L05_SOT89 -> MC79L06F-TP; MPN (none) -> MC79L06F-TP
Connections:
- net GND: now also D11.2 (A), E1.1, E2.1, GD1.2, NT2.2; no longer TP13.1
- net return_kelvin: now also E2.2
- net at R12.1, R13.2, TP8.1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: now also GD1.1
- net at F1.2, FB5.1, TP14.1: now also D11.1 (K)
- net at R1.1, TP11.1: now also E1.2
- new net: NT2.1, TP13.1
Other:
- note added: "Connections for coil PCB trace fuse and spark gap as protection for arc to coil"
- note removed: "Connections for coil"
- moved on the sheet: C20, C21, C22, C23, C24, C25, C26, C27, C28, C29, C30, C31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

Commit message: next design revision
Parts:
- removed C18: 47n, Capacitor_SMD:C_0805_2012Metric, symbol Device:C
- removed C24, C26, C32: 47u, Capacitor_Tantalum_SMD:CP_EIA-3528-15_AVX-H, symbol Device:C_Polarized
- removed C33, C34, C8: 0.47u, Capacitor_SMD:C_0603_1608Metric, symbol Device:C
- removed D10: LED_Dual_KAKA, wbraun_smd:LED_WP934MD, symbol Device:LED_Dual_KAKA
- removed D6, D7: 1N4148, Diode_SMD:D_SOD-323F, symbol Device:D
- removed D8, D9: MM3Z7V5B, Diode_SMD:D_SOD-323F, symbol Device:D_Zener
- removed J2: RFShield_TwoPieces, wbraun_smd:Masach_Tech_MS288-10F, symbol Device:RFShield_TwoPieces
- removed NT2: NetTie_2, NetTie:NetTie-2_SMD_Pad0.5mm, symbol Device:NetTie_2
- removed Q1: MMBT3906, wbraun_smd:SOT-23, symbol Device:Q_PNP_BEC
- removed Q2: MMBT3904, wbraun_smd:SOT-23, symbol Device:Q_NPN_BEC
- removed R22, R23, R27: 47k, Resistor_SMD:R_0603_1608Metric, symbol Device:R
- removed R24, R29: 22k, Resistor_SMD:R_0603_1608Metric, symbol Device:R
- removed R26: 1M, Resistor_SMD:R_0603_1608Metric, symbol Device:R
- removed R28, R30: 4.7k, Resistor_SMD:R_0603_1608Metric, symbol Device:R
- removed R31, R32: 0.1, Resistor_SMD:R_0603_1608Metric, symbol Device:R
- removed TP1, TP10, TP2, TP3, TP5, TP7, TP8, TP9: TestPoint, wbraun_smd:THM_MINI, symbol Connector:TestPoint
- removed TP13: TestPoint, TestPoint:TestPoint_Pad_4.0x4.0mm, symbol Connector:TestPoint
- added C2, C3: 10u, Capacitor_SMD:C_1206_3216Metric, symbol Device:C
- added C4: DNP, Capacitor_SMD:C_0603_1608Metric, symbol Device:C
- added D6: LTST-S220KGKT, wbraun_smd:LED-T1-RIGHT-ANGLE_4.6x4.4mm, symbol Device:LED
- added J1, J2, J3, J4: ECT81800C036, wbraun_smd:Shield_Clip_ECT81800C036, symbol Device:RFShield_OnePiece
- C10: value 22p -> DNP; MPN CL10C220JB81PNC -> (none)
- C11: value 8-40p -> 12-60p; footprint Capacitor_SMD:C_Trimmer_Voltronics_JZ -> wbraun_smd:C_Trimmer_GKG_6mm; MPN JZ400 -> GKG60015
- C12, C13, C5, C6: JLC_MPN (none) -> C1623; MPN CL10B474KA8NFNC -> CL10B474KA8NNNC
- C14, C22: JLC_MPN (none) -> C1664
- C15: footprint Capacitor_SMD:C_0805_2012Metric -> Capacitor_SMD:C_1206_3216Metric; JLC_MPN (none) -> C21812; MPN C3216C0G1H473J115AA -> GRM31M5C1H473JA01L
- C17: value 47n -> DNP; footprint Capacitor_SMD:C_0805_2012Metric -> Capacitor_SMD:C_0603_1608Metric; MPN C3216C0G1H473J115AA -> (none)
- C19: value 22p -> 10p; JLC_MPN (none) -> C1634; MPN CL10C220JB81PNC -> CL10C100JB8NNNC
- C20, C23, C25, C27, C28, C29, C30, C31: JLC_MPN (none) -> C13585; MPN CL31A106KAHNNNE -> CL31A106KBHNNNE
- C7: value 0.47u -> 10u; footprint Capacitor_SMD:C_0603_1608Metric -> Capacitor_SMD:C_1206_3216Metric; JLC_MPN (none) -> C13585; MPN CL10B474KA8NFNC -> CL31A106KBHNNNE
- C9: value 150p -> 100p; JLC_MPN (none) -> C107033; MPN CL10C151JB8NFNC -> CC0603JRNPO0BN101
- D1, D2: JLC_MPN (none) -> C2128
- D11: value SMAJ6.0A-13-F -> P6SMB6.8CA/TR13; footprint Diode_SMD:D_SMA -> Diode_SMD:D_SMB; JLC_MPN (none) -> C78395; MPN SMAJ6.0A-13-F -> P6SMB6.8CA/TR13
- D3, D4, D5: value PD3S140-7 -> BAT760-7; footprint wbraun_smd:D_POWERDI323 -> Diode_SMD:D_SOD-323; JLC_MPN (none) -> C191023; MPN PD3S140-7 -> BAT760-7
- F1: JLC_MPN (none) -> C163512
- FB3, FB4, FB5: JLC_MPN (none) -> C1015
- GD1: JLC_MPN (none) -> C522627
- J7: JLC_MPN (none) -> C530662
- J8: JLC_MPN (none) -> C498173
- L1: JLC_MPN (none) -> C136244
- L2: JLC_MPN (none) -> C91596
- R1: footprint Resistor_SMD:R_1206_3216Metric -> Resistor_SMD:R_0603_1608Metric; JLC_MPN (none) -> C23182; MPN RMCF1206FT47R0 -> (none)
- R10: value 220 -> 470; JLC_MPN (none) -> C23179; MPN RMCF0603FT220R -> (none)
- R11, R12: value 2k -> 470; JLC_MPN (none) -> C23179; MPN RMCF0603FT2K00 -> (none)
- R13: value 47 -> 100; JLC_MPN (none) -> C17901; MPN RMCF1206FT47R0 -> (none)
- R14: JLC_MPN (none) -> C21189
- R15, R18: value 75k -> 82k; JLC_MPN (none) -> C23254; MPN RMCF0603FT75K0 -> (none)
- R16: value 13.3k -> 13k; JLC_MPN (none) -> C22797; MPN RMCF0603FT13K3 -> (none)
- R19: value 0 -> DNP; MPN RMCF0805ZT0R00 -> (none)
- R2: value 4.7k -> 22k; JLC_MPN (none) -> C31850; MPN RMCF0603FT4K70 -> RMCF0603FG22K0
- R20: value 2k -> DNP; MPN RMCF0603FT2K00 -> (none)
- R21: value 2k -> 100; footprint Resistor_SMD:R_0603_1608Metric -> Resistor_SMD:R_1206_3216Metric; JLC_MPN (none) -> C17901; MPN RMCF0603FT2K00 -> (none)
- R25: value 1M -> 4.7k; JLC_MPN (none) -> C23162; MPN RMCF0603FG1M00 -> RMCF0603FT4K70
- R3: value 10k -> 8.2k; JLC_MPN (none) -> C25981; MPN RMCF0603FT10K0 -> (none)
- R4, R7: value 47k -> 22k; JLC_MPN (none) -> C31850; MPN RMCF0603FT47K0 -> RMCF0603FG22K0
- R5: JLC_MPN (none) -> C23032
- R6: value 22k -> DNP; MPN RMCF0603FG22K0 -> (none)
- R8: value 2k -> 10k; JLC_MPN (none) -> C25804; MPN RMCF0603FT2K00 -> (none)
- R9: value 10k -> 2k; JLC_MPN (none) -> C22975; MPN RMCF0603FT10K0 -> (none)
- RV1: footprint wbraun_smd:TRIMMER_PVG3A -> Potentiometer_SMD:Potentiometer_Bourns_3314G_Vertical; JLC_MPN (none) -> C52238; MPN PVG3A201C01R00 -> 3314G-1-201E
- U1: JLC_MPN (none) -> C17271
- U2: JLC_MPN (none) -> C408904
- U3: JLC_MPN (none) -> C468235
- U4: JLC_MPN (none) -> C81357
- U5: JLC_MPN (none) -> C8619
Connections:
- net GND: now also C16.1, C7.2, R20.2, R7.2, RV1.1, U1.3 (+), C2.2, C3.1, J1.1 (Shield), J2.1 (Shield), J3.1 (Shield), J4.1 (Shield); no longer C16.2, C7.1, R8.1, RV1.3, U1.5 (+)
- net VBUS: now also C7.1
- net VDD: now also C30.1, U4.1 (OUT); no longer C7.2
- net VDD_unreg: now also C2.1
- net VSS: now also C31.2, U5.3 (VO), D6.1 (K)
- net VSS_unreg: now also C3.2
- net int_out: now also R10.2, C4.1; no longer C17.1, R7.2
- net at C15.1, R4.2: now also U1.7; no longer U1.1
- net out: now reaches R12.1, R13.2, U2.7
- net out: now also C17.1, R21.2, R8.2; no longer GD1.1
- net at R20.1: now also C17.2
- net at R25.1: now also D6.2 (A)
- net at J7.1 (In), R13.1: now also GD1.1, R21.1
- net at U1.6 (-): now also C15.2, R7.1; no longer U1.7
- net at R5.1: now also RV1.3; no longer RV1.1
- net int_fb: now reaches C14.1, R2.1, R5.2, U2.2 (-)
- new net: C16.2, R8.1, R9.2, U1.5 (+)
- new net: C4.2, R6.1
- new net: U1.1, U1.2 (-)
Other:
- note added: "Connector Subs: 0732515490 73251-2200 RF2-49B-T-00-50-G-HDW < cheapest JLC: C530662"
- note added: "LCSC Subs: AD8022ARZ-REEL7 OPA211AIDR LT6231CS8#PBF AD8066ARZ-R7 (?) For low speed amp: BA4558F-E2 OPA2197IDR OPA2188AIDR (best) COS2227USR (cheaper)"
- note added: "OPA2188AIDR through JLC assembly"
- note added: "Regulates at 9V sub BAT760-7 diode for lower capacitance"
- note added: "similar JLC stocked var cap is JML06-1-20P"
- note removed: "+/- 8V to LDO"
- note removed: "Connector Subs: 0732515490 73251-2200 RF2-49B-T-00-50-G-HDW < cheapest"
- note removed: "Overload (red)"
- note removed: "Power (green)"
- note removed: "Simple overload detect circuitry"
- note removed: "Trigger when int_out gets to +-3V Vbe + Vdiode + Vzener"
- note removed: "shield for power supply"
- moved on the sheet: C19, C20, C21, C22, C23, C25, C27, C28, C29, C30, C31, D3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

Commit message: design revision
Parts:
- removed FB5: FerriteBead_Small, Inductor_SMD:L_0805_2012Metric, symbol Device:FerriteBead_Small
- removed L2: DLW5BTM142SQ2L, wbraun_smd:L_CommonModeChoke_Murata_DLW5BTM, symbol Device:L_Ferrite_Coupled
- removed R19: DNP, Resistor_SMD:R_0805_2012Metric, symbol Device:R
- removed R20: DNP, Resistor_SMD:R_0603_1608Metric, symbol Device:R
- removed R21: 100, Resistor_SMD:R_1206_3216Metric, symbol Device:R
- removed TP14: TestPoint, wbraun_smd:THM_MINI, symbol Connector:TestPoint
- added C18, C8: 0.47u, Capacitor_SMD:C_0603_1608Metric, symbol Device:C
- added C24: 10u, Capacitor_SMD:C_1206_3216Metric, symbol Device:C
- added H1: MountingHole, wbraun_smd:beefield_logo_small, symbol Mechanical:MountingHole
- added L2, L3: 6.8u, Inductor_SMD:L_1210_3225Metric, symbol Device:L
- added U6: B0505S-1WR3, wbraun_smd:Converter_DCDC_1W_Isolated_Short, symbol Regulator_Switching:CRE1S0505SC
- C17: value DNP -> 1n; footprint Capacitor_SMD:C_0603_1608Metric -> Capacitor_SMD:C_1206_3216Metric
- C4: value DNP -> 10u; footprint Capacitor_SMD:C_0603_1608Metric -> Capacitor_SMD:C_1206_3216Metric; JLC_MPN (none) -> C13585; MPN (none) -> CL31A106KBHNNNE
- D6: value LTST-S220KGKT -> WP934CB/GD
- R13: value 100 -> 47; JLC_MPN C17901 -> (none)
- R6: value DNP -> 47; JLC_MPN (none) -> C23182
Connections:
- net GND: now also C17.2, C18.2, C24.2, U6.3 (-VOUT); no longer D11.2 (A), R6.2
- net VBUS: now also C24.1, L3.2
- net int_out: no longer C4.1
- net out: no longer C17.1
- net at J8.1 (VBUS): now also F1.1
- net USB_GND: now reaches J8.4 (GND)
- net USB_GND: now also C17.1, C4.2, D11.2 (A), J8.5 (Shield), C8.2, U6.1 (-VIN)
- net at C1.1, C10.1, C11.1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: now also R6.1; no longer U2.3 (+)
- net USB_PWR: now reaches D11.1 (K), F1.2
- net USB_PWR: now also C4.1, L2.1
- new net: C8.1, L2.2, U6.2 (+VIN)
- new net: C18.1, L3.1, U6.4 (+VOUT)
- new net: R6.2, U2.3 (+)
Other:
- moved on the sheet: D11, F1

Commit message: pcb sent to production
Parts:
- removed C20, C23, C24, C25, C27: 10u, Capacitor_SMD:C_1206_3216Metric, symbol Device:C
- removed C21: DNP, Capacitor_SMD:C_0603_1608Metric, symbol Device:C
- removed C22: 330p, Capacitor_SMD:C_0603_1608Metric, symbol Device:C
- removed D3, D4, D5: BAT760-7, Diode_SMD:D_SOD-323, symbol Device:D_Schottky
- removed FB3, FB4: FerriteBead_Small, Inductor_SMD:L_0805_2012Metric, symbol Device:FerriteBead_Small
- removed J1, J2, J3, J4: ECT81800C036, wbraun_smd:Shield_Clip_ECT81800C036, symbol Device:RFShield_OnePiece
- removed L1: 10u, wbraun_smd:L_VLCF4020, symbol Device:L
- removed R15, R18: 82k, Resistor_SMD:R_0603_1608Metric, symbol Device:R
- removed R16: 13k, Resistor_SMD:R_0603_1608Metric, symbol Device:R
- removed R17: DNP, Resistor_SMD:R_0805_2012Metric, symbol Device:R
- removed U3: LMR62014XMF, Package_TO_SOT_SMD:SOT-23-5, symbol Regulator_Switching:LMR62014XMF
- removed U6: B0505S-1WR3, wbraun_smd:Converter_DCDC_1W_Isolated_Short, symbol Regulator_Switching:CRE1S0505SC
- added FB1, FB2: FerriteBead_Small, Inductor_SMD:L_0805_2012Metric, symbol Device:FerriteBead_Small
- added H2, H3, H4, H5: MountingHole, wbraun_smd:JLC_TOOLING_HOLE, symbol Mechanical:MountingHole
- added L1: DLW5BTM102SQ2L, wbraun_smd:L_CommonModeChoke_Murata_DLW5BTM, symbol Device:L_Ferrite_Coupled
- added L4: 10u, Inductor_SMD:L_1210_3225Metric, symbol Device:L
- added PS1: A0509S-2WR3, Converter_DCDC:Converter_DCDC_XP_POWER-IHxxxxS_THT, symbol Converter_DCDC:IH0503S
- C14: MPN CL10C330JB8NNNC -> (none)
- C17: JLC_MPN (none) -> C9196
- C18, C8: value 0.47u -> 10u; footprint Capacitor_SMD:C_0603_1608Metric -> Capacitor_SMD:C_1206_3216Metric; JLC_MPN C1623 -> C13585; MPN CL10B474KA8NNNC -> CL31A106KBHNNNE
- L2, L3: value 6.8u -> 10u; JLC_MPN C250230 -> C21764; MPN NLCV32T-6R8M-EF -> NLCV32T-100K-EFD
- NT1: value NetTie_2 -> DNP
- R13: JLC_MPN (none) -> C17969
- R3: value 8.2k -> 22k; JLC_MPN C25981 -> C31850; MPN (none) -> RMCF0603FG22K0
- R5: value 365 -> 360; JLC_MPN C23032 -> C25194; MPN RC0603FR-07365RL -> (none)
- R9: value 2k -> 470; JLC_MPN C22975 -> C23179
- TP11, TP12, TP4, TP6: value TestPoint -> DNP
- U4: JLC_MPN C81357 -> C81358
Connections:
- net GND: now also C18.1, C3.2, C7.1, C8.2, PS1.5 (0V); no longer C17.2, C18.2, C2.2, C3.1, C7.2
- net USB_GND: now also C2.2, L1.4, PS1.2 (-Vin); no longer C8.2, J8.4 (GND), J8.5 (Shield)
- net VDD_unreg: now also C28.1, U4.3 (IN), FB1.2; no longer C2.1
- net VSS_unreg: now also C29.2, U5.2 (VI), FB2.2; no longer C3.2
- net at C8.1: now also L3.2, FB1.1; no longer L2.2
- net at L3.1: now also C3.1, PS1.6 (+Vout); no longer C18.1
- net at F1.1: now also L1.2; no longer J8.1 (VBUS)
- removed net VBUS: C7.1, L3.2
- new net: C17.2, C7.2, L4.1, PS1.4 (-Vout)
- new net: C18.2, FB2.1, L4.2
- new net: C2.1, L2.2, PS1.1 (+Vin)
- new net: J8.1 (VBUS), L1.1
- new net: J8.4 (GND), J8.5 (Shield), L1.3
Other:
- note added: "10mV worst case DC offset"
- note added: "AD8022ARZ-REEL7 through JLC assembly"
- note added: "Assembly fixture holes"
- note added: "placeholder for logo"
- note removed: "Regulates at 9V sub BAT760-7 diode for lower capacitance"
- moved on the sheet: C28, C29, C30, C31, C4, D11, F1, H1, L3, U4, U5

Commit message: next revision
Parts:
- removed R11, R12: 470, Resistor_SMD:R_0603_1608Metric, symbol Device:R
- removed TP11, TP12: DNP, TestPoint:TestPoint_Pad_4.0x4.0mm, symbol Connector:TestPoint
- added C22: 47p, Capacitor_SMD:C_0603_1608Metric, symbol Device:C
- added J2: Conn_Coaxial, Connector_Coaxial:U.FL_Hirose_U.FL-R-SMT-1_Vertical, symbol Connector:Conn_Coaxial
- added R13: 1.2k, Resistor_SMD:R_0603_1608Metric, symbol Device:R
- added R14: 169, Resistor_SMD:R_0603_1608Metric, symbol Device:R
- added R15: 220, Resistor_SMD:R_0603_1608Metric, symbol Device:R
- added RV2: 200, Potentiometer_SMD:Potentiometer_Bourns_3314G_Vertical, symbol Device:R_Potentiometer_Trim
- C10: renamed from C1; value DNP -> 10p; JLC_MPN (none) -> C1634; MPN (none) -> CL10C100JB8NNNC
- C11: value 12-60p -> DNP; MPN GKG60015 -> (none)
- C6: renamed from C9; value 100p -> 180p; JLC_MPN C107033 -> C527047; MPN CC0603JRNPO0BN101 -> CC0603FRNPO9BN181
- C8: renamed from C10; value DNP -> 10p; JLC_MPN (none) -> C1634; MPN (none) -> CL10C100JB8NNNC
- F1: footprint Fuse:Fuse_1206_3216Metric -> Fuse:Fuse_0603_1608Metric; JLC_MPN C163512 -> C206991; MPN 0ZCJ0050FF2G -> 0467.750NRHF
- J3: renamed from J7; JLC_MPN C530662 -> C1509208; MPN RF2-49B-T-00-50-G-HDW -> (none)
- L1: value DLW5BTM102SQ2L -> DLW5BTM142SQ2L; JLC_MPN C70478 -> C91596; MPN (none) -> DLW5BTM142SQ2L
- L2, L3, L4: value 10u -> 6.8u; JLC_MPN C21764 -> C250230; MPN NLCV32T-100K-EFD -> NLCV32T-6R8M-EF
- PS1: JLC_MPN C2827996 -> (none)
- R3: renamed from R5; value 360 -> 430; JLC_MPN C25194 -> C23170
- R8: renamed from R10; value 470 -> 220; JLC_MPN C23179 -> C22962
- U2: JLC_MPN C408904 -> (none)
- renumbered C5 to C1, C3 to C12, C7 to C13, C8 to C15, C18 to C16, C15 to C17, C19 to C18, C16 to C19, C6 to C2, C28 to C20, C29 to C21, C30 to C23, C31 to C24, C12 to C3, C13 to C4, C4 to C5, C2 to C7, C17 to C9, D11 to D1, D1 to D2, D2 to D3, D6 to D4, J8 to J1, R8 to R10, R9 to R12, R13 to R16, R25 to R17, R6 to R2, R2 to R4, R3 to R5, R14 to R6, R4 to R7, R7 to R9, TP4 to TP1, TP6 to TP2, U4 to U3, U5 to U4
Connections:
- net GND: now also C10.2, C11.1, C6.2, C8.2, C22.2, R15.2
- net out: now also R14.1
- net return_kelvin: now also J2.2 (Ext); no longer C10.2, C11.2, C6.2, C8.2
- net at C10.1, C6.1, C8.1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: now also C11.2; no longer C11.1
- net at U2.6 (-): now also R13.1, RV2.2
- net at E1.2, R1.1: now also J2.1 (In)
- new net: C22.1, R13.2
- new net: R14.2, RV2.3
- new net: R15.1, RV2.1
Other:
- note added: "Nominal gain of 2x Trim between 1.4x to 2.6x"
- note removed: "similar JLC stocked var cap is JML06-1-20P"
- moved on the sheet: C1, C10, C11, C12, C13, C14, C15, C16, C17, C18, C19, C2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

Commit message: first public release
Parts:
- removed C11: DNP, wbraun_smd:C_Trimmer_GKG_6mm, symbol Device:C_Trim
- removed E2: SparkGap, wbraun_smd:Spark_Gap, symbol Device:SparkGap
- removed NT1: DNP, NetTie:NetTie-2_SMD_Pad0.5mm, symbol Device:NetTie_2
- added C11: DNP, Capacitor_SMD:C_0603_1608Metric, symbol Device:C
- added J3, J4, J5, J6: Conn_01x01_Female, wbraun_smd:CLIP_ECT81800C036, symbol Connector:Conn_01x01_Female
- added R2, R3: 4.7, Resistor_SMD:R_0603_1608Metric, symbol Device:R
- added R5: 47, Resistor_SMD:R_0603_1608Metric, symbol Device:R
- C10: renamed from C9; MPN (none) -> 1206B102K202NT
- C14: MPN (none) -> CL10C331JB8NNNC
- C5: renamed from C6; value 180p -> 68p; JLC_MPN C527047 -> C28262; MPN CC0603FRNPO9BN181 -> CL10C680JB8NNNC
- C7: renamed from C8; value 10p -> 68p; JLC_MPN C1634 -> C28262; MPN CL10C100JB8NNNC -> CL10C680JB8NNNC
- C9: renamed from C10; value 10p -> 68p; JLC_MPN C1634 -> C28262; MPN CL10C100JB8NNNC -> CL10C680JB8NNNC
- D3: renamed from D1; value P6SMB6.8CA/TR13 -> 6.8V
- D4: JLC_MPN C2929606 -> C2929607
- GD1: value GDT_2Pin -> 75V
- J1: renamed from J2; value Conn_Coaxial -> U.FL; MPN (none) -> U.FL-R-SMT-1(10)
- J7: renamed from J3; value Conn_Coaxial -> SMA; MPN (none) -> RF2-49B-T-00-50-G-HDW
- PS1: value A0509S-2WR3 -> A0509S-1WR3; JLC_MPN (none) -> C131900; MPN (none) -> A0509S-1WR3
- R1: MPN (none) -> RC0603FR-0747RL
- R11: renamed from R8; MPN (none) -> RC0603FR-07220RL
- R13: renamed from R10; MPN (none) -> RC0603FR-0710KL
- R14: renamed from R12; MPN (none) -> RC0603FR-07470RL
- R15: renamed from R13; MPN (none) -> RC0603FR-071K2L
- R16: renamed from R14; MPN (none) -> RC0603FR-07169RL
- R17: renamed from R15; MPN (none) -> RC0603FR-07220RL
- R19: renamed from R17; value 4.7k -> 2.2k; JLC_MPN C23162 -> C4190; MPN RMCF0603FT4K70 -> RC0603FR-072K2L
- R4: renamed from R2; value 47 -> 4.7; JLC_MPN C23182 -> C23164; MPN (none) -> RC0603JR-074R7L
- R6: renamed from R3; MPN (none) -> RC0603FR-07430RL
- U1: value TLV2172 -> OPA2188; MPN TLV2172IDR -> OPA2188AIDR
- U2: JLC_MPN (none) -> C2059808
- renumbered C5 to C6, C7 to C8, D2 to D1, D3 to D2, J1 to J2, R7 to R10, R9 to R12, R16 to R18, R4 to R7, R5 to R8, R6 to R9
Connections:
- net return_kelvin is gone; now on net GND: J1.2 (Ext)
- net GND: now also C11.1, J3.1 (Pin_1), J4.1 (Pin_1), J5.1 (Pin_1), J6.1 (Pin_1)
- net at C9.1, D1.2 (A), D2.1 (K)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: now also R3.2; no longer C5.1, C7.1, R1.2
- net at R4.2: now also C11.2, R5.1; no longer U2.3 (+)
- new net: C5.1, R1.2, R2.1
- new net: C7.1, R2.2, R3.1
- new net: R5.2, U2.3 (+)
Other:
- note added: "Coil input"
- note added: "EMI Shield Clips Mate with 30x20mm can P/N: S01-30200500"
- note added: "Filters out of band EMI"
- note added: "Gain peaking to compensate for coil HF attenuation"
- note added: "Integrator"
- note added: "Output Buffer"
- note added: "PCB trace fuse and spark gap as protection for coil flashover"
- note added: "Protection in case of coil flashover"
- note added: "Right angle THT SMA 6.5mm center height off PCB"
- note added: "Servo HP filter"
- note added: "Test Points"
- note added: "trim crossover"
- note removed: "10mV worst case DC offset"
- note removed: "AD8022ARZ-REEL7 through JLC assembly"
- note removed: "Connections for coil PCB trace fuse and spark gap as protection for arc to coil"
- note removed: "Connector Subs: 0732515490 73251-2200 RF2-49B-T-00-50-G-HDW < cheapest JLC: C530662"
- note removed: "LCSC Subs: AD8022ARZ-REEL7 OPA211AIDR LT6231CS8#PBF AD8066ARZ-R7 (?) For low speed amp: BA4558F-E2 OPA2197IDR OPA2188AIDR (best) COS2227USR (cheaper)"
- note removed: "OPA2188AIDR through JLC assembly"
- moved on the sheet: C1, C10, C12, C13, C14, C15, C16, C17, C18, C19, C2, C20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
